File: Amp.kicad_sch (KiCad schematic)
At the start: 17 parts, among them U1 TL431DBZ, U2 LM358

Commit message: Version V1.0 Ordered
Parts:
- removed R4: 360, Resistor_SMD:R_0805_2012Metric, symbol Device:R
- removed unit 3 of U2
- added J2: Conn_01x01_Pin, Connector_PinHeader_2.54mm:PinHeader_1x01_P2.54mm_Vertical, symbol Connector:Conn_01x01_Pin
- added R1: 120, Resistor_SMD:R_0805_2012Metric, symbol Device:R
- RV1: now in the parts list
Connections:
- net B2: now also J2.1 (Pin_1), R1.2
- net VCC: now also R1.1
