File: StrainGuageAmpV1_0.kicad_pcb (KiCad board)
At the start: 2 copper layers, 50.8 x 34.9 mm, 45 parts, among them J1 Conn_01x04_Pin, J3 Screw_Terminal_01x04, U1 TL431DBZ, U2 LM358, U3 TL431DBZ, U4 LM358

Commit message: Version V1.0 Ordered
Parts:
- removed R15, R4: 360, Resistor_SMD:R_0805_2012Metric
- added J2: Conn_01x01_Pin, Connector_PinHeader_2.54mm:PinHeader_1x01_P2.54mm_Vertical, F.Cu at (194.3, 32.4)
- added J4: Conn_01x01_Pin, Connector_PinHeader_2.54mm:PinHeader_1x01_P2.54mm_Vertical, F.Cu at (183.1, 59.1)
- added R1: 120, Resistor_SMD:R_0805_2012Metric, F.Cu at (190.2, 40.0)
- added R11: 120, Resistor_SMD:R_0805_2012Metric, F.Cu at (190.2, 55.0)
Connections:
- U2 pad 8: /Amp1/VFF -> VCC
- U4 pad 8: /Amp2/VFF -> VCC
Routing:
- net VCC: track 17.5 -> 51.1 mm, vias 0 -> 2
- net /Amp1/VFF: track 60.0 -> 68.6 mm
- net /Amp2/VFF: track 59.7 -> 65.3 mm
- net GND: vias 19 -> 20
Other:
- board text added: "VFF1"
- board text added: "VFF2"
