File: StrainGuageAmpV1_0.kicad_sch (KiCad schematic)
At the start: 11 parts, among them J1 Conn_01x04_Pin, J3 Screw_Terminal_01x04

Commit message: Version V1.0 Ordered
Parts:
- added U2, U4: LM358, Package_SO:SOIC-8_3.9x4.9mm_P1.27mm, symbol Amplifier_Operational:LM358
- H1, H2, H3, H4, J1: now not fitted
Connections:
- net GND: now also U2.4 (V-), U4.4 (V-)
- net VCC: now also U2.8 (V+), U4.8 (V+)
